File: ebaz_adaptor.kicad_pcb (KiCad board)
At the start: 2 copper layers, 100 x 68 mm, 53 parts, among them J1 data-1, J10 pmod 1, J11 pmod 2, J12 camera, J2 data-2, J3 data-3, J4 +12V pwr, J5 Z-Turn Extension, J6 Alinx HDMI/ETH module, J7 ADC module 2-ch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

Commit message: add screenshots
Other:
- board text added: "locked"
- board text removed: "A20"
- board text removed: "B19"
- board text removed: "C20"
- board text removed: "D20"
- board text removed: "H17"
- board text removed: "H18"
